Commit message: Cleaned up unnecessary packages and modifications for Velodyne to publish topics and visualize in RViz

File: jackal_description/urdf/accessories/vlp16_mount.urdf.xacro (robot description, xacro)
@@ -87,5 +87,5 @@
         <origin xyz="0 0 ${height}" rpy="0 0 0" />
       </joint>
-      <xacro:VLP-16 parent="${prefix}_vlp16_plate" topic="${topic}">
+      <xacro:VLP-16 parent="${prefix}_vlp16_plate" name="velodyne" topic="/velodyne_points" hz="10" samples="440" gpu="true">
         <origin xyz="0 0 0" rpy="0 0 0" />
       </xacro:VLP-16>

File: jackal_description/urdf/jackal.urdf.xacro (robot description, xacro)
@@ -232,4 +232,9 @@
     <xacro:outdoornav_sensors outdoornav_configuration="$(arg outdoornav_configuration)" />
   </xacro:if>
+  <!-- VLP-16 -->
+  <!-- <xacro:include filename="$(find velodyne_description)/urdf/VLP-16.urdf.xacro"/>
+  <xacro:VLP-16 parent="base_link" name="velodyne" topic="/velodyne_points" hz="10" samples="440" gpu="true">
+    <origin xyz="0 0 0.4" rpy="0 0 0" />
+  </xacro:VLP-16> -->
   <!-- Optional custom includes. -->
   <xacro:include filename="$(optenv JACKAL_URDF_EXTRAS empty.urdf)" />
